File: SUSTAINA-Power-Monitor-Module/design/Power-Monitor-Module.sch (EAGLE design)
At the start: 21 parts, among them IC1 INA226, P1 2X5P, P2 2X5P, P3 1X4P

Commit message: Corrected the silk printing and via processing method
Other:
- note added: "May 25, 2024"
- note removed: "May 1, 2024"
Changed lines of the file:
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@@
 <text x="5.08" y="132.08" size="5.08" layer="97" align="top-left">Pinhedders</text>
 <text x="5.08" y="205.74" size="5.08" layer="97" align="top-left">Current-shunt and power monitor</text>
-<text x="185.42" y="5.08" size="5.08" layer="94" ratio="10" align="center-left">May 1, 2024</text>
+<text x="185.42" y="5.08" size="5.08" layer="94" ratio="10" align="center-left">May 25, 2024</text>
 <text x="185.42" y="25.4" size="5.08" layer="94" ratio="10" align="center-left">SUSTAINA Power Monitor Module</text>
 <text x="269.24" y="15.24" size="5.08" layer="94" ratio="10" align="center-left">3.0</text>
