File: SUSTAINA-PMX-Control-Board/design/SUSTAINA-PMX-Control-Board.brd (EAGLE design)
At the start: 67 x 45 mm, 20 parts, among them M1 USB-TO-QUAD-RS-485-CONV-MODUL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

Commit message: Add mass-produced version of PMX-Control-Board
Parts:
- added C1: 0.1u, rcl:C0603
- added C2: 10u, rcl:C0603
- added CH6, CH7, CH8, CH9: B2B-PH-K-S(LF)(SN), JST-PH:B2B-PH-K-S(LF)(SN)
- added U$19, U$7: (no value), buzzard_labels:DC_FAN
- added U$6: (no value), buzzard_labels:PMX
- added U1: LM2937IMP-12NOPB, LM2937IMP-12NOPB:SOT-223
- U$1, U$2: device buzzard_labels:DESIGNED_BY_MASATO_KUBOTERA_ON_MAY_1 -> buzzard_labels:DESIGNED_BY_MASATO_KUBOTERA_ON_JUNE_1
- moved U$1 39.4 mm to (30.5, -16.5), turned to 90 degrees
- moved U$12 34.4 mm to (27.9, -13.3), turned to 90 degrees
- moved U$5 20.2 mm to (-21.0, -13.3), turned to 270 degrees
Connections:
- new net +12V: C2.1, CH6.2, CH7.2, CH8.2, CH9.2, U1.3
- net +PWR: now also C1.1, U1.1
- net GND: now also C1.2, C2.2, CH6.1, CH7.1, CH8.1, CH9.1, U1.2
Routing:
- net GND: track 0.00 -> 12.4 mm, vias 0 -> 3
- net +PWR: track 4.79 -> 0.00 mm
- net A-DP: track 49.9 -> 48.7 mm
- net A-DM: track 51.1 -> 50.0 mm
- added copper zone on layer 1, net +12V
- added copper zone on layer 1, net +PWR
- added copper zone on layer 16, net GND
- removed copper zone on layer 16, net +PWR
- removed copper zone on layer 1, net GND
